Commit message: backup before robot reset

File: erwhi_description/urdf/erwhi.urdf (robot description, URDF)
Before this commit: robot erwhi, 3 links, 2 joints
Links:
- added link camera_link; collision box size=0.01 0.14 0.02; visual box size=0.01 0.14 0.02
- added link imu_link; collision box size=0.02 0.03 0.005; visual box size=0.02 0.03 0.005
Joints:
- added joint camera_joint: type fixed, parent base_link, child camera_link, origin xyz=0.045 0.00 0.094 rpy=0.0 0.0 0.0
- added joint imu_joint: type fixed, parent base_link, child imu_link, origin xyz=-0.025 0.05 0.11 rpy=0.0 0.0 0.0

Commit message: update

File: erwhi_description/urdf/erwhi.urdf (robot description, URDF)
Before this commit: robot erwhi, 5 links, 4 joints
Links:
- added link base_laser; visual cylinder length=0.06 radius=0.035
- link base_link: geometry visual cylinder length=0.06 radius=0.07
- link left_wheel: geometry collision cylinder length=0.01 radius=0.0365125; visual cylinder length=0.01 radius=0.0365125
- link right_wheel: geometry collision cylinder length=0.01 radius=0.0365125; visual cylinder length=0.01 radius=0.0365125
Joints:
- added joint base_link_to_base_laser: type fixed, parent base_link, child base_laser, origin xyz=0 0 0.15 rpy=0 0 -1.5708
- joint left_joint: origin xyz=0 0.07 0.05 rpy=1.57075 0.0 0.0 -> xyz=0 0.07 0.0365125 rpy=1.57075 0.0 0.0
- joint right_joint: origin xyz=0 -0.07 0.05 rpy=1.57075 0.0 0.0 -> xyz=0 -0.07 0.0365125 rpy=1.57075 0.0 0.0
